File: cart.kicad_pcb (KiCad board)
At the start: 2 copper layers, 66 x 40 mm, 7 parts, among them P1 CONN_SMS, U1 27C256

Commit message: re-run autorouter
Parts:
- moved C2 4.45 mm to (169.5, 90.2)
- moved U1 1.09 mm to (123.8, 92.1)
- moved C1 0.48 mm to (117.5, 73.0)
Routing:
- net GND: track 14.1 -> 87.5 mm
- net OE: track 49.9 -> 67.7 mm
- net /d5: track 28.6 -> 39.5 mm
- net /d7: track 36.9 -> 43.7 mm
- net /d3: track 28.0 -> 34.0 mm, vias 1 -> 0
- net /a10: track 45.0 -> 48.3 mm
- net /d4: track 36.9 -> 33.9 mm, vias 0 -> 1
- net /a7: track 18.1 -> 15.3 mm
- net /d6: track 29.7 -> 32.4 mm, vias 0 -> 1
- net /d1: track 12.8 -> 11.7 mm
- net /d0: track 11.8 -> 10.6 mm
- net /a0: track 11.8 -> 10.6 mm
- net /d2: track 12.8 -> 11.7 mm
- net /a1: track 11.3 -> 10.3 mm
- net /a4: track 12.3 -> 11.3 mm
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